Commit message: CableBlock

File: ur3_sim_description/urdf/gripper.xacro (robot description, xacro)
@@ -503,8 +503,25 @@
     </joint>
     <joint name="gripper" type="fixed">
-      <origin xyz="0.00875 0.022171 0.0814375" rpy="${3.141/2.0} 0.0 ${-3.141/2.0}" />zzz
+      <origin xyz="0.00875 0.022171 0.0814375" rpy="${3.141/2.0} 0.0 ${-3.141/2.0}" />
       <parent link="tool0" />
       <child link="base_bottom" />
     </joint>
+    <link name="cable_block">
+      <visual>
+        <geometry>
+          <mesh filename="package://ur3_sim_description/meshes/gripper/CableBlock.dae" scale="0.001 0.001 0.001"/>
+        </geometry>
+      </visual>
+      <collision>
+        <geometry>
+          <mesh filename="package://ur3_sim_description/meshes/gripper/CableBlock.dae" scale="0.001 0.001 0.001"/>
+        </geometry>
+      </collision>
+    </link>
+    <joint name="cable_block_joint" type="fixed">
+      <origin xyz="0.0 0.0 0.0" rpy="0.0 0.0 ${3.141}" />
+      <parent link="base_bottom" />
+      <child link="cable_block" />
+    </joint>
   </xacro:macro>
 </robot>

Commit message: Update gripper.xacro

File: ur3_sim_description/urdf/gripper.xacro (robot description, xacro)
@@ -94,5 +94,5 @@
       <axis xyz="0 0 -1"/>
       <origin xyz="0.0 0 0.0"/>
-      <limit effort="1000.0" lower="-2.0" upper="2.0" velocity="0.5"/>
+      <limit effort="1000.0" lower="-2.0" upper="2.0" velocity="1.5"/>
     </joint>
     <link name="right_gear">
@@ -127,5 +127,5 @@
       <axis xyz="0 0 1"/>
       <origin xyz="0.044341 0 0.0"/>
-      <limit effort="1000.0" lower="-2.0" upper="2.0" velocity="0.5"/>
+      <limit effort="1000.0" lower="-2.0" upper="2.0" velocity="1.5"/>
       <mimic joint="left_gear_joint" multiplier="1" offset="0" />
     </joint>
@@ -158,5 +158,5 @@
       <axis xyz="0 0 1"/>
       <origin xyz="0.050137 0 0.0"/>
-      <limit effort="1000.0" lower="-2.0" upper="2.0" velocity="0.5"/>
+      <limit effort="1000.0" lower="-2.0" upper="2.0" velocity="1.5"/>
       <mimic joint="left_gear_joint" multiplier="-1" offset="0" />
     </joint>
@@ -189,5 +189,5 @@
       <axis xyz="0 0 1"/>
       <origin xyz="-0.050137 0 0.0"/>
-      <limit effort="1000.0" lower="-2.0" upper="2.0" velocity="0.5"/>
+      <limit effort="1000.0" lower="-2.0" upper="2.0" velocity="1.5"/>
       <mimic joint="left_gear_joint" multiplier="1" offset="0" />
     </joint>
@@ -219,5 +219,5 @@
       <axis xyz="0 0 1"/>
       <origin xyz="0.050137  0 0.0"/>
-     <limit effort="1000.0" lower="-2.0" upper="2.0" velocity="0.5"/>
+     <limit effort="1000.0" lower="-2.0" upper="2.0" velocity="1.5"/>
       <mimic joint="left_gear_joint" multiplier="-1" offset="0" />
     </joint>
@@ -249,5 +249,5 @@
       <axis xyz="0 0 1"/>
       <origin xyz="-0.050137 0 0.0"/>
-      <limit effort="1000.0" lower="-2.0" upper="2.0" velocity="0.5"/>
+      <limit effort="1000.0" lower="-2.0" upper="2.0" velocity="1.5"/>
       <mimic joint="left_gear_joint" multiplier="1" offset="0" />
     </joint>
@@ -341,5 +341,5 @@
       <axis xyz="0 0 1"/>
         <origin xyz="0.01 0.033 0.0"/>
-      <limit effort="1000.0" lower="-2.0" upper="2.0" velocity="0.5"/>
+      <limit effort="1000.0" lower="-2.0" upper="2.0" velocity="1.5"/>
       <mimic joint="left_gear_joint" multiplier="-1" offset="0" />
     </joint>
@@ -375,5 +375,5 @@
       <axis xyz="0 0 1"/>
         <origin xyz="0.034341 0.033 0.0"/>
-      <limit effort="1000.0" lower="-2.0" upper="2.0" velocity="0.5"/>
+      <limit effort="1000.0" lower="-2.0" upper="2.0" velocity="1.5"/>
       <mimic joint="left_gear_joint" multiplier="1" offset="0" />
     </joint>
@@ -438,5 +438,5 @@
       <axis xyz="0 0 1"/>
       <origin xyz="0.01 0.033 0.0"/>
-      <limit effort="1000.0" lower="-2.0" upper="2.0" velocity="0.5"/>
+      <limit effort="1000.0" lower="-2.0" upper="2.0" velocity="1.5"/>
       <mimic joint="left_gear_joint" multiplier="-1" offset="0" />
     </joint>
@@ -472,5 +472,5 @@
       <axis xyz="0 0 1"/>
       <origin xyz="0.034341 0.033 0.0"/>
-      <limit effort="1000.0" lower="-2.0" upper="2.0" velocity="0.5"/>
+      <limit effort="1000.0" lower="-2.0" upper="2.0" velocity="1.5"/>
       <mimic joint="left_gear_joint" multiplier="1" offset="0" />
     </joint>
